File: Hardware/Kicad files.kicad_pcb (KiCad board)
At the start: 2 copper layers, 89 x 58.5 mm, 13 parts, among them SW1 SW_Push, SW2 SW_Push, SW3 SW_Push, SW4 SW_Push, SW5 RotaryEncoder, U1 XIAO-RP2040-DIP

Commit message: Added Stickers on PCB
Parts:
- added G***: LOGO, LOGO, F.Cu at (81.9, 70.8)
- added G***: LOGO, LOGO, B.Cu at (79.0, 72.0)
- added G***: LOGO, LOGO, B.Cu at (92.5, 86.0)
